File: kicad/boards/led_panel/led_panel_3/led_panel_3.kicad_sch (KiCad schematic)
At the start: 2 parts

Commit message: feat: complete circuit designs for all ALU components
* Designed all gate modules: AND, OR, NOT, NAND, NOR, XOR (1-bit and 8-bit variants)

* Completed multiplexer hierarchy: 2:1, 4:1, and 8:1 8-bit muxes

* Finalized add_sub board schematic and LED panel designs

* Added new board modules: flags, main_control, main_logic

* Updated Logisim top-level ALU circuit

* Note: KiCad directory path errors to be resolved next (iCloud sync issue), then begin PCB routing
Parts:
- added D102: LED22, LED_THT:LED_D3.0mm, symbol Device:LED
- added D103: LED21, LED_THT:LED_D3.0mm, symbol Device:LED
- added D104: LED23, LED_THT:LED_D3.0mm, symbol Device:LED
- added R102, R103, R104: 300, Resistor_SMD:R_0805_2012Metric, symbol Device:R
- D101: value LED -> LED20
Connections:
- net GND: now also D102.1 (K), D103.1 (K), D104.1 (K)
- new net: D103.2 (A), R103.1
- new net: D102.2 (A), R102.1
- new net: D104.2 (A), R104.1
- new net EQ_FL: R103.2
- new net GREAT_FL: R104.2
- new net LESS_FL: R102.2
