File: kicad/modules/gates/gate_inv/gate_inv_8bit/gate_inv_8bit.kicad_sch (KiCad schematic)
At the start: 0 parts

Commit message: feat: complete circuit designs for all ALU components
* Designed all gate modules: AND, OR, NOT, NAND, NOR, XOR (1-bit and 8-bit variants)

* Completed multiplexer hierarchy: 2:1, 4:1, and 8:1 8-bit muxes

* Finalized add_sub board schematic and LED panel designs

* Added new board modules: flags, main_control, main_logic

* Updated Logisim top-level ALU circuit

* Note: KiCad directory path errors to be resolved next (iCloud sync issue), then begin PCB routing
Other:
- sheet inv1: file ../gate_inv_1bit/gate_inv_1bit.kicad_sch -> ../../modules/gates/gate_inv/gate_inv_1bit/gate_inv_1bit.kicad_sch
- sheet inv2: file ../gate_inv_1bit/gate_inv_1bit.kicad_sch -> ../../modules/gates/gate_inv/gate_inv_1bit/gate_inv_1bit.kicad_sch
- sheet inv3: file ../gate_inv_1bit/gate_inv_1bit.kicad_sch -> ../../modules/gates/gate_inv/gate_inv_1bit/gate_inv_1bit.kicad_sch
- sheet inv4: file ../gate_inv_1bit/gate_inv_1bit.kicad_sch -> ../../modules/gates/gate_inv/gate_inv_1bit/gate_inv_1bit.kicad_sch
- sheet inv5: file ../gate_inv_1bit/gate_inv_1bit.kicad_sch -> ../../modules/gates/gate_inv/gate_inv_1bit/gate_inv_1bit.kicad_sch
- sheet inv6: file ../gate_inv_1bit/gate_inv_1bit.kicad_sch -> ../../modules/gates/gate_inv/gate_inv_1bit/gate_inv_1bit.kicad_sch
- sheet inv7: file ../gate_inv_1bit/gate_inv_1bit.kicad_sch -> ../../modules/gates/gate_inv/gate_inv_1bit/gate_inv_1bit.kicad_sch
- sheet inv8: file ../gate_inv_1bit/gate_inv_1bit.kicad_sch -> ../../modules/gates/gate_inv/gate_inv_1bit/gate_inv_1bit.kicad_sch
Changed lines of the file:
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@@
 			)
 		)
-		(property "Sheetfile" "../gate_inv_1bit/gate_inv_1bit.kicad_sch"
+		(property "Sheetfile" "../../modules/gates/gate_inv/gate_inv_1bit/gate_inv_1bit.kicad_sch"
 			(at 41.91 57.7346 0)
 			(effects
@@
 				(path "/d141fce1-7092-474f-ac13-21228438d92c"
 					(page "4")
+				)
+			)
+			(project ""
+				(path "/724c0b0c-29d0-4c6a-be9f-fdb8b4c646fb"
+					(page "")
+				)
+			)
+			(project "main_logic"
+				(path "/9c59990f-2fe5-4da7-bc07-d03b445b1465/724c0b0c-29d0-4c6a-be9f-fdb8b4c646fb"
+					(page "24")
+				)
+			)
+			(project ""
+				(path "/0f98840f-83e1-46ff-ab4b-366905a86376"
+					(page "")
 				)
 			)
@@
 			)
 		)
-		(property "Sheetfile" "../gate_inv_1bit/gate_inv_1bit.kicad_sch"
+		(property "Sheetfile" "../../modules/gates/gate_inv/gate_inv_1bit/gate_inv_1bit.kicad_sch"
 			(at 41.91 121.2346 0)
 			(effects
@@
 				(path "/d141fce1-7092-474f-ac13-21228438d92c"
 					(page "9")
+				)
+			)
+			(project ""
+				(path "/724c0b0c-29d0-4c6a-be9f-fdb8b4c646fb"
+					(page "")
+				)
+			)
+			(project "main_logic"
+				(path "/9c59990f-2fe5-4da7-bc07-d03b445b1465/724c0b0c-29d0-4c6a-be9f-fdb8b4c646fb"
+					(page "30")
+				)
+			)
+			(project ""
+				(path "/0f98840f-83e1-46ff-ab4b-366905a86376"
+					(page "")
 				)
 			)
@@
 			)
 		)
-		(property "Sheetfile" "../gate_inv_1bit/gate_inv_1bit.kicad_sch"
+		(property "Sheetfile" "../../modules/gates/gate_inv/gate_inv_1bit/gate_inv_1bit.kicad_sch"
 			(at 41.91 95.8346 0)
 			(effects
@@
 				(path "/d141fce1-7092-474f-ac13-21228438d92c"
 					(page "7")
+				)
+			)
+			(project ""
+				(path "/724c0b0c-29d0-4c6a-be9f-fdb8b4c646fb"
+					(page "")
+				)
+			)
+			(project "main_logic"
+				(path "/9c59990f-2fe5-4da7-bc07-d03b445b1465/724c0b0c-29d0-4c6a-be9f-fdb8b4c646fb"
+					(page "28")
+				)
+			)
+			(project ""
+				(path "/0f98840f-83e1-46ff-ab4b-366905a86376"
+					(page "")
 				)
 			)
@@
 			)
 		)
-		(property "Sheetfile" "../gate_inv_1bit/gate_inv_1bit.kicad_sch"
+		(property "Sheetfile" "../../modules/gates/gate_inv/gate_inv_1bit/gate_inv_1bit.kicad_sch"
 			(at 41.91 32.3346 0)
 			(effects
@@
 				(path "/d141fce1-7092-474f-ac13-21228438d92c"
 					(page "2")
+				)
+			)
+			(project ""
+				(path "/724c0b0c-29d0-4c6a-be9f-fdb8b4c646fb"
+					(page "")
+				)
+			)
+			(project "main_logic"
+				(path "/9c59990f-2fe5-4da7-bc07-d03b445b1465/724c0b0c-29d0-4c6a-be9f-fdb8b4c646fb"
+					(page "22")
+				)
+			)
+			(project ""
+				(path "/0f98840f-83e1-46ff-ab4b-366905a86376"
+					(page "")
 				)
 			)
@@
 			)
 		)
-		(property "Sheetfile" "../gate_inv_1bit/gate_inv_1bit.kicad_sch"
+		(property "Sheetfile" "../../modules/gates/gate_inv/gate_inv_1bit/gate_inv_1bit.kicad_sch"
 			(at 41.91 70.4346 0)
 			(effects
@@
 				(path "/d141fce1-7092-474f-ac13-21228438d92c"
 					(page "5")
+				)
+			)
+			(project ""
+				(path "/724c0b0c-29d0-4c6a-be9f-fdb8b4c646fb"
+					(page "")
+				)
+			)
+			(project "main_logic"
+				(path "/9c59990f-2fe5-4da7-bc07-d03b445b1465/724c0b0c-29d0-4c6a-be9f-fdb8b4c646fb"
+					(page "26")
+				)
+			)
+			(project ""
+				(path "/0f98840f-83e1-46ff-ab4b-366905a86376"
+					(page "")
 				)
 			)
@@
 			)
 		)
-		(property "Sheetfile" "../gate_inv_1bit/gate_inv_1bit.kicad_sch"
+		(property "Sheetfile" "../../modules/gates/gate_inv/gate_inv_1bit/gate_inv_1bit.kicad_sch"
 			(at 41.91 45.0346 0)
 			(effects
@@
 				(path "/d141fce1-7092-474f-ac13-21228438d92c"
 					(page "3")
+				)
+			)
+			(project ""
+				(path "/724c0b0c-29d0-4c6a-be9f-fdb8b4c646fb"
+					(page "")
+				)
+			)
+			(project "main_logic"
+				(path "/9c59990f-2fe5-4da7-bc07-d03b445b1465/724c0b0c-29d0-4c6a-be9f-fdb8b4c646fb"
+					(page "23")
+				)
+			)
+			(project ""
+				(path "/0f98840f-83e1-46ff-ab4b-366905a86376"
+					(page "")
 				)
 			)
@@
 			)
 		)
-		(property "Sheetfile" "../gate_inv_1bit/gate_inv_1bit.kicad_sch"
+		(property "Sheetfile" "../../modules/gates/gate_inv/gate_inv_1bit/gate_inv_1bit.kicad_sch"
 			(at 41.91 83.1346 0)
 			(effects
@@
 				(path "/d141fce1-7092-474f-ac13-21228438d92c"
 					(page "6")
+				)
+			)
+			(project ""
+				(path "/724c0b0c-29d0-4c6a-be9f-fdb8b4c646fb"
+					(page "")
+				)
+			)
+			(project "main_logic"
+				(path "/9c59990f-2fe5-4da7-bc07-d03b445b1465/724c0b0c-29d0-4c6a-be9f-fdb8b4c646fb"
+					(page "27")
+				)
+			)
+			(project ""
+				(path "/0f98840f-83e1-46ff-ab4b-366905a86376"
+					(page "")
 				)
 			)
@@
 			)
 		)
-		(property "Sheetfile" "../gate_inv_1bit/gate_inv_1bit.kicad_sch"
+		(property "Sheetfile" "../../modules/gates/gate_inv/gate_inv_1bit/gate_inv_1bit.kicad_sch"
 			(at 41.91 108.5346 0)
 			(effects
@@
 				)
 			)
-		)
-	)
-	(sheet_instances
-		(path "/"
-			(page "1")
-		)
-	)
-	(embedded_fonts no)
+			(project ""
+				(path "/724c0b0c-29d0-4c6a-be9f-fdb8b4c646fb"
+					(page "")
+				)
+			)
+			(project "main_logic"
+				(path "/9c59990f-2fe5-4da7-bc07-d03b445b1465/724c0b0c-29d0-4c6a-be9f-fdb8b4c646fb"
+					(page "29")
+				)
+			)
+			(project ""
+				(path "/0f98840f-83e1-46ff-ab4b-366905a86376"
+					(page "")
+				)
+			)
+		)
+	)
 )

Commit message: Fix KiCad file paths and complete core circuit design
- Fixed file path errors across all KiCad schematics and projects
- Completed core circuit designs:
  * Adder and subtractor modules (adder2, adder8)
  * LED panels (led_panel_1) with display circuits
  * Flag LED circuits for status indicators
  * All dependent logic gate modules (AND, OR, NOT, NAND, NOR, XOR)
  * All multiplexer modules (2:1, 4:1, 8:1, 8-bit)
  * Main control board schematics
  * Flags board schematics
- Updated .gitignore to exclude KiCad backups, cache files, and lock files
- Ready for pin placement and routing of control buses, power rails, and inter-board signals
Other:
- sheet inv1: file ../../modules/gates/gate_inv/gate_inv_1bit/gate_inv_1bit.kicad_sch -> ../gate_inv_1bit/gate_inv_1bit.kicad_sch
- sheet inv2: file ../../modules/gates/gate_inv/gate_inv_1bit/gate_inv_1bit.kicad_sch -> ../gate_inv_1bit/gate_inv_1bit.kicad_sch
- sheet inv3: file ../../modules/gates/gate_inv/gate_inv_1bit/gate_inv_1bit.kicad_sch -> ../gate_inv_1bit/gate_inv_1bit.kicad_sch
- sheet inv4: file ../../modules/gates/gate_inv/gate_inv_1bit/gate_inv_1bit.kicad_sch -> ../gate_inv_1bit/gate_inv_1bit.kicad_sch
- sheet inv5: file ../../modules/gates/gate_inv/gate_inv_1bit/gate_inv_1bit.kicad_sch -> ../gate_inv_1bit/gate_inv_1bit.kicad_sch
- sheet inv6: file ../../modules/gates/gate_inv/gate_inv_1bit/gate_inv_1bit.kicad_sch -> ../gate_inv_1bit/gate_inv_1bit.kicad_sch
- sheet inv7: file ../../modules/gates/gate_inv/gate_inv_1bit/gate_inv_1bit.kicad_sch -> ../gate_inv_1bit/gate_inv_1bit.kicad_sch
- sheet inv8: file ../../modules/gates/gate_inv/gate_inv_1bit/gate_inv_1bit.kicad_sch -> ../gate_inv_1bit/gate_inv_1bit.kicad_sch
