File: kicad/modules/gates/gate_nand/gate_nand_2in_8bit/gate_nand_2in_8bit.kicad_sch (KiCad schematic)
At the start: 0 parts

Commit message: feat: complete circuit designs for all ALU components
* Designed all gate modules: AND, OR, NOT, NAND, NOR, XOR (1-bit and 8-bit variants)

* Completed multiplexer hierarchy: 2:1, 4:1, and 8:1 8-bit muxes

* Finalized add_sub board schematic and LED panel designs

* Added new board modules: flags, main_control, main_logic

* Updated Logisim top-level ALU circuit

* Note: KiCad directory path errors to be resolved next (iCloud sync issue), then begin PCB routing
Other:
- sheet nand2_1: file ../gate_nand_2in/gate_nand_2in.kicad_sch -> ../../modules/gates/gate_nand/gate_nand_2in/gate_nand_2in.kicad_sch
- sheet nand2_2: file ../gate_nand_2in/gate_nand_2in.kicad_sch -> ../../modules/gates/gate_nand/gate_nand_2in/gate_nand_2in.kicad_sch
- sheet nand2_3: file ../gate_nand_2in/gate_nand_2in.kicad_sch -> ../../modules/gates/gate_nand/gate_nand_2in/gate_nand_2in.kicad_sch
- sheet nand2_4: file ../gate_nand_2in/gate_nand_2in.kicad_sch -> ../../modules/gates/gate_nand/gate_nand_2in/gate_nand_2in.kicad_sch
- sheet nand2_5: file ../gate_nand_2in/gate_nand_2in.kicad_sch -> ../../modules/gates/gate_nand/gate_nand_2in/gate_nand_2in.kicad_sch
- sheet nand2_6: file ../gate_nand_2in/gate_nand_2in.kicad_sch -> ../../modules/gates/gate_nand/gate_nand_2in/gate_nand_2in.kicad_sch
- sheet nand2_7: file ../gate_nand_2in/gate_nand_2in.kicad_sch -> ../../modules/gates/gate_nand/gate_nand_2in/gate_nand_2in.kicad_sch
- sheet nand2_8: file ../gate_nand_2in/gate_nand_2in.kicad_sch -> ../../modules/gates/gate_nand/gate_nand_2in/gate_nand_2in.kicad_sch
Changed lines of the file:
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@@
 			)
 		)
-		(property "Sheetfile" "../gate_nand_2in/gate_nand_2in.kicad_sch"
+		(property "Sheetfile" "../../modules/gates/gate_nand/gate_nand_2in/gate_nand_2in.kicad_sch"
 			(at 34.29 50.1146 0)
 			(effects
@@
 			(project "gate_nand_2in_8bit"
 				(path "/5db9410b-1a15-448c-89b3-091faadf870e"
+					(page "3")
+				)
+			)
+			(project ""
+				(path "/3114c630-b5bb-4706-a171-8ab374ad8acb"
+					(page "#")
+				)
+			)
+			(project "main_logic"
+				(path "/9c59990f-2fe5-4da7-bc07-d03b445b1465/3114c630-b5bb-4706-a171-8ab374ad8acb"
 					(page "3")
 				)
@@
 			)
 		)
-		(property "Sheetfile" "../gate_nand_2in/gate_nand_2in.kicad_sch"
+		(property "Sheetfile" "../../modules/gates/gate_nand/gate_nand_2in/gate_nand_2in.kicad_sch"
 			(at 34.29 132.6646 0)
 			(effects
@@
 			(project "gate_nand_2in_8bit"
 				(path "/5db9410b-1a15-448c-89b3-091faadf870e"
+					(page "8")
+				)
+			)
+			(project ""
+				(path "/3114c630-b5bb-4706-a171-8ab374ad8acb"
+					(page "#")
+				)
+			)
+			(project "main_logic"
+				(path "/9c59990f-2fe5-4da7-bc07-d03b445b1465/3114c630-b5bb-4706-a171-8ab374ad8acb"
 					(page "8")
 				)
@@
 			)
 		)
-		(property "Sheetfile" "../gate_nand_2in/gate_nand_2in.kicad_sch"
+		(property "Sheetfile" "../../modules/gates/gate_nand/gate_nand_2in/gate_nand_2in.kicad_sch"
 			(at 34.29 116.1546 0)
 			(effects
@@
 			(project "gate_nand_2in_8bit"
 				(path "/5db9410b-1a15-448c-89b3-091faadf870e"
+					(page "7")
+				)
+			)
+			(project ""
+				(path "/3114c630-b5bb-4706-a171-8ab374ad8acb"
+					(page "#")
+				)
+			)
+			(project "main_logic"
+				(path "/9c59990f-2fe5-4da7-bc07-d03b445b1465/3114c630-b5bb-4706-a171-8ab374ad8acb"
 					(page "7")
 				)
@@
 			)
 		)
-		(property "Sheetfile" "../gate_nand_2in/gate_nand_2in.kicad_sch"
+		(property "Sheetfile" "../../modules/gates/gate_nand/gate_nand_2in/gate_nand_2in.kicad_sch"
 			(at 34.29 83.1346 0)
 			(effects
@@
 			(project "gate_nand_2in_8bit"
 				(path "/5db9410b-1a15-448c-89b3-091faadf870e"
+					(page "5")
+				)
+			)
+			(project ""
+				(path "/3114c630-b5bb-4706-a171-8ab374ad8acb"
+					(page "#")
+				)
+			)
+			(project "main_logic"
+				(path "/9c59990f-2fe5-4da7-bc07-d03b445b1465/3114c630-b5bb-4706-a171-8ab374ad8acb"
 					(page "5")
 				)
@@
 			)
 		)
-		(property "Sheetfile" "../gate_nand_2in/gate_nand_2in.kicad_sch"
+		(property "Sheetfile" "../../modules/gates/gate_nand/gate_nand_2in/gate_nand_2in.kicad_sch"
 			(at 34.29 149.1746 0)
 			(effects
@@
 			(project "gate_nand_2in_8bit"
 				(path "/5db9410b-1a15-448c-89b3-091faadf870e"
+					(page "9")
+				)
+			)
+			(project ""
+				(path "/3114c630-b5bb-4706-a171-8ab374ad8acb"
+					(page "#")
+				)
+			)
+			(project "main_logic"
+				(path "/9c59990f-2fe5-4da7-bc07-d03b445b1465/3114c630-b5bb-4706-a171-8ab374ad8acb"
 					(page "9")
 				)
@@
 			)
 		)
-		(property "Sheetfile" "../gate_nand_2in/gate_nand_2in.kicad_sch"
+		(property "Sheetfile" "../../modules/gates/gate_nand/gate_nand_2in/gate_nand_2in.kicad_sch"
 			(at 34.29 99.6446 0)
 			(effects
@@
 			(project "gate_nand_2in_8bit"
 				(path "/5db9410b-1a15-448c-89b3-091faadf870e"
+					(page "6")
+				)
+			)
+			(project ""
+				(path "/3114c630-b5bb-4706-a171-8ab374ad8acb"
+					(page "#")
+				)
+			)
+			(project "main_logic"
+				(path "/9c59990f-2fe5-4da7-bc07-d03b445b1465/3114c630-b5bb-4706-a171-8ab374ad8acb"
 					(page "6")
 				)
@@
 			)
 		)
-		(property "Sheetfile" "../gate_nand_2in/gate_nand_2in.kicad_sch"
+		(property "Sheetfile" "../../modules/gates/gate_nand/gate_nand_2in/gate_nand_2in.kicad_sch"
 			(at 34.29 66.6246 0)
 			(effects
@@
 			(project "gate_nand_2in_8bit"
 				(path "/5db9410b-1a15-448c-89b3-091faadf870e"
+					(page "4")
+				)
+			)
+			(project ""
+				(path "/3114c630-b5bb-4706-a171-8ab374ad8acb"
+					(page "#")
+				)
+			)
+			(project "main_logic"
+				(path "/9c59990f-2fe5-4da7-bc07-d03b445b1465/3114c630-b5bb-4706-a171-8ab374ad8acb"
 					(page "4")
 				)
@@
 			)
 		)
-		(property "Sheetfile" "../gate_nand_2in/gate_nand_2in.kicad_sch"
+		(property "Sheetfile" "../../modules/gates/gate_nand/gate_nand_2in/gate_nand_2in.kicad_sch"
 			(at 34.29 33.6046 0)
 			(effects
@@
 				)
 			)
-		)
-	)
-	(sheet_instances
-		(path "/"
-			(page "1")
-		)
-	)
-	(embedded_fonts no)
+			(project ""
+				(path "/3114c630-b5bb-4706-a171-8ab374ad8acb"
+					(page "#")
+				)
+			)
+			(project "main_logic"
+				(path "/9c59990f-2fe5-4da7-bc07-d03b445b1465/3114c630-b5bb-4706-a171-8ab374ad8acb"
+					(page "2")
+				)
+			)
+		)
+	)
 )

Commit message: Fix KiCad file paths and complete core circuit design
- Fixed file path errors across all KiCad schematics and projects
- Completed core circuit designs:
  * Adder and subtractor modules (adder2, adder8)
  * LED panels (led_panel_1) with display circuits
  * Flag LED circuits for status indicators
  * All dependent logic gate modules (AND, OR, NOT, NAND, NOR, XOR)
  * All multiplexer modules (2:1, 4:1, 8:1, 8-bit)
  * Main control board schematics
  * Flags board schematics
- Updated .gitignore to exclude KiCad backups, cache files, and lock files
- Ready for pin placement and routing of control buses, power rails, and inter-board signals
Other:
- sheet nand2_1: file ../../modules/gates/gate_nand/gate_nand_2in/gate_nand_2in.kicad_sch -> ../gate_nand_2in/gate_nand_2in.kicad_sch
- sheet nand2_2: file ../../modules/gates/gate_nand/gate_nand_2in/gate_nand_2in.kicad_sch -> ../gate_nand_2in/gate_nand_2in.kicad_sch
- sheet nand2_3: file ../../modules/gates/gate_nand/gate_nand_2in/gate_nand_2in.kicad_sch -> ../gate_nand_2in/gate_nand_2in.kicad_sch
- sheet nand2_4: file ../../modules/gates/gate_nand/gate_nand_2in/gate_nand_2in.kicad_sch -> ../gate_nand_2in/gate_nand_2in.kicad_sch
- sheet nand2_5: file ../../modules/gates/gate_nand/gate_nand_2in/gate_nand_2in.kicad_sch -> ../gate_nand_2in/gate_nand_2in.kicad_sch
- sheet nand2_6: file ../../modules/gates/gate_nand/gate_nand_2in/gate_nand_2in.kicad_sch -> ../gate_nand_2in/gate_nand_2in.kicad_sch
- sheet nand2_7: file ../../modules/gates/gate_nand/gate_nand_2in/gate_nand_2in.kicad_sch -> ../gate_nand_2in/gate_nand_2in.kicad_sch
- sheet nand2_8: file ../../modules/gates/gate_nand/gate_nand_2in/gate_nand_2in.kicad_sch -> ../gate_nand_2in/gate_nand_2in.kicad_sch
