File: kicad/modules/gates/gate_nor/gate_nor_2in_8bit/gate_nor_2in_8bit.kicad_sch (KiCad schematic)
At the start: 0 parts

Commit message: feat: complete circuit designs for all ALU components
* Designed all gate modules: AND, OR, NOT, NAND, NOR, XOR (1-bit and 8-bit variants)

* Completed multiplexer hierarchy: 2:1, 4:1, and 8:1 8-bit muxes

* Finalized add_sub board schematic and LED panel designs

* Added new board modules: flags, main_control, main_logic

* Updated Logisim top-level ALU circuit

* Note: KiCad directory path errors to be resolved next (iCloud sync issue), then begin PCB routing
Other:
- sheet 2nor1: file ../gate_nor_2in_1bit/gate_nor_2in.kicad_sch -> ../../modules/gates/gate_nor/gate_nor_2in_1bit/gate_nor_2in.kicad_sch
- sheet 2nor2: file ../gate_nor_2in_1bit/gate_nor_2in.kicad_sch -> ../../modules/gates/gate_nor/gate_nor_2in_1bit/gate_nor_2in.kicad_sch
- sheet 2nor3: file ../gate_nor_2in_1bit/gate_nor_2in.kicad_sch -> ../../modules/gates/gate_nor/gate_nor_2in_1bit/gate_nor_2in.kicad_sch
- sheet 2nor4: file ../gate_nor_2in_1bit/gate_nor_2in.kicad_sch -> ../../modules/gates/gate_nor/gate_nor_2in_1bit/gate_nor_2in.kicad_sch
- sheet 2nor5: file ../gate_nor_2in_1bit/gate_nor_2in.kicad_sch -> ../../modules/gates/gate_nor/gate_nor_2in_1bit/gate_nor_2in.kicad_sch
- sheet 2nor6: file ../gate_nor_2in_1bit/gate_nor_2in.kicad_sch -> ../../modules/gates/gate_nor/gate_nor_2in_1bit/gate_nor_2in.kicad_sch
- sheet 2nor7: file ../gate_nor_2in_1bit/gate_nor_2in.kicad_sch -> ../../modules/gates/gate_nor/gate_nor_2in_1bit/gate_nor_2in.kicad_sch
- sheet 2nor8: file ../gate_nor_2in_1bit/gate_nor_2in.kicad_sch -> ../../modules/gates/gate_nor/gate_nor_2in_1bit/gate_nor_2in.kicad_sch
Changed lines of the file:
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@@
 			)
 		)
-		(property "Sheetfile" "../gate_nor_2in_1bit/gate_nor_2in.kicad_sch"
+		(property "Sheetfile" "../../modules/gates/gate_nor/gate_nor_2in_1bit/gate_nor_2in.kicad_sch"
 			(at 62.23 84.4046 0)
 			(effects
@@
 				(path "/1dc696ed-d35e-495d-aad0-47f49dae0428"
 					(page "5")
+				)
+			)
+			(project ""
+				(path "/b0b24703-6682-42ff-bfe8-9b2bd3fa2617"
+					(page "#")
+				)
+			)
+			(project "main_logic"
+				(path "/9c59990f-2fe5-4da7-bc07-d03b445b1465/b0b24703-6682-42ff-bfe8-9b2bd3fa2617"
+					(page "13")
 				)
 			)
@@
 			)
 		)
-		(property "Sheetfile" "../gate_nor_2in_1bit/gate_nor_2in.kicad_sch"
+		(property "Sheetfile" "../../modules/gates/gate_nor/gate_nor_2in_1bit/gate_nor_2in.kicad_sch"
 			(at 62.23 132.6646 0)
 			(effects
@@
 				(path "/1dc696ed-d35e-495d-aad0-47f49dae0428"
 					(page "8")
+				)
+			)
+			(project ""
+				(path "/b0b24703-6682-42ff-bfe8-9b2bd3fa2617"
+					(page "#")
+				)
+			)
+			(project "main_logic"
+				(path "/9c59990f-2fe5-4da7-bc07-d03b445b1465/b0b24703-6682-42ff-bfe8-9b2bd3fa2617"
+					(page "16")
 				)
 			)
@@
 			)
 		)
-		(property "Sheetfile" "../gate_nor_2in_1bit/gate_nor_2in.kicad_sch"
+		(property "Sheetfile" "../../modules/gates/gate_nor/gate_nor_2in_1bit/gate_nor_2in.kicad_sch"
 			(at 62.23 149.1746 0)
 			(effects
@@
 				(path "/1dc696ed-d35e-495d-aad0-47f49dae0428"
 					(page "9")
+				)
+			)
+			(project ""
+				(path "/b0b24703-6682-42ff-bfe8-9b2bd3fa2617"
+					(page "#")
+				)
+			)
+			(project "main_logic"
+				(path "/9c59990f-2fe5-4da7-bc07-d03b445b1465/b0b24703-6682-42ff-bfe8-9b2bd3fa2617"
+					(page "17")
 				)
 			)
@@
 			)
 		)
-		(property "Sheetfile" "../gate_nor_2in_1bit/gate_nor_2in.kicad_sch"
+		(property "Sheetfile" "../../modules/gates/gate_nor/gate_nor_2in_1bit/gate_nor_2in.kicad_sch"
 			(at 62.23 117.4246 0)
 			(effects
@@
 				(path "/1dc696ed-d35e-495d-aad0-47f49dae0428"
 					(page "7")
+				)
+			)
+			(project ""
+				(path "/b0b24703-6682-42ff-bfe8-9b2bd3fa2617"
+					(page "#")
+				)
+			)
+			(project "main_logic"
+				(path "/9c59990f-2fe5-4da7-bc07-d03b445b1465/b0b24703-6682-42ff-bfe8-9b2bd3fa2617"
+					(page "15")
 				)
 			)
@@
 			)
 		)
-		(property "Sheetfile" "../gate_nor_2in_1bit/gate_nor_2in.kicad_sch"
+		(property "Sheetfile" "../../modules/gates/gate_nor/gate_nor_2in_1bit/gate_nor_2in.kicad_sch"
 			(at 62.23 34.8746 0)
 			(effects
@@
 				(path "/1dc696ed-d35e-495d-aad0-47f49dae0428"
 					(page "2")
+				)
+			)
+			(project ""
+				(path "/b0b24703-6682-42ff-bfe8-9b2bd3fa2617"
+					(page "#")
+				)
+			)
+			(project "main_logic"
+				(path "/9c59990f-2fe5-4da7-bc07-d03b445b1465/b0b24703-6682-42ff-bfe8-9b2bd3fa2617"
+					(page "10")
 				)
 			)
@@
 			)
 		)
-		(property "Sheetfile" "../gate_nor_2in_1bit/gate_nor_2in.kicad_sch"
+		(property "Sheetfile" "../../modules/gates/gate_nor/gate_nor_2in_1bit/gate_nor_2in.kicad_sch"
 			(at 62.23 51.3846 0)
 			(effects
@@
 				(path "/1dc696ed-d35e-495d-aad0-47f49dae0428"
 					(page "3")
+				)
+			)
+			(project ""
+				(path "/b0b24703-6682-42ff-bfe8-9b2bd3fa2617"
+					(page "#")
+				)
+			)
+			(project "main_logic"
+				(path "/9c59990f-2fe5-4da7-bc07-d03b445b1465/b0b24703-6682-42ff-bfe8-9b2bd3fa2617"
+					(page "11")
 				)
 			)
@@
 			)
 		)
-		(property "Sheetfile" "../gate_nor_2in_1bit/gate_nor_2in.kicad_sch"
+		(property "Sheetfile" "../../modules/gates/gate_nor/gate_nor_2in_1bit/gate_nor_2in.kicad_sch"
 			(at 62.23 100.9146 0)
 			(effects
@@
 				(path "/1dc696ed-d35e-495d-aad0-47f49dae0428"
 					(page "6")
+				)
+			)
+			(project ""
+				(path "/b0b24703-6682-42ff-bfe8-9b2bd3fa2617"
+					(page "#")
+				)
+			)
+			(project "main_logic"
+				(path "/9c59990f-2fe5-4da7-bc07-d03b445b1465/b0b24703-6682-42ff-bfe8-9b2bd3fa2617"
+					(page "14")
 				)
 			)
@@
 			)
 		)
-		(property "Sheetfile" "../gate_nor_2in_1bit/gate_nor_2in.kicad_sch"
+		(property "Sheetfile" "../../modules/gates/gate_nor/gate_nor_2in_1bit/gate_nor_2in.kicad_sch"
 			(at 62.23 67.8946 0)
 			(effects
@@
 				)
 			)
-		)
-	)
-	(sheet_instances
-		(path "/"
-			(page "1")
-		)
-	)
-	(embedded_fonts no)
+			(project ""
+				(path "/b0b24703-6682-42ff-bfe8-9b2bd3fa2617"
+					(page "#")
+				)
+			)
+			(project "main_logic"
+				(path "/9c59990f-2fe5-4da7-bc07-d03b445b1465/b0b24703-6682-42ff-bfe8-9b2bd3fa2617"
+					(page "12")
+				)
+			)
+		)
+	)
 )

Commit message: Fix KiCad file paths and complete core circuit design
- Fixed file path errors across all KiCad schematics and projects
- Completed core circuit designs:
  * Adder and subtractor modules (adder2, adder8)
  * LED panels (led_panel_1) with display circuits
  * Flag LED circuits for status indicators
  * All dependent logic gate modules (AND, OR, NOT, NAND, NOR, XOR)
  * All multiplexer modules (2:1, 4:1, 8:1, 8-bit)
  * Main control board schematics
  * Flags board schematics
- Updated .gitignore to exclude KiCad backups, cache files, and lock files
- Ready for pin placement and routing of control buses, power rails, and inter-board signals
Other:
- sheet 2nor1: file ../../modules/gates/gate_nor/gate_nor_2in_1bit/gate_nor_2in.kicad_sch -> ../gate_nor_2in_1bit/gate_nor_2in.kicad_sch
- sheet 2nor2: file ../../modules/gates/gate_nor/gate_nor_2in_1bit/gate_nor_2in.kicad_sch -> ../gate_nor_2in_1bit/gate_nor_2in.kicad_sch
- sheet 2nor3: file ../../modules/gates/gate_nor/gate_nor_2in_1bit/gate_nor_2in.kicad_sch -> ../gate_nor_2in_1bit/gate_nor_2in.kicad_sch
- sheet 2nor4: file ../../modules/gates/gate_nor/gate_nor_2in_1bit/gate_nor_2in.kicad_sch -> ../gate_nor_2in_1bit/gate_nor_2in.kicad_sch
- sheet 2nor5: file ../../modules/gates/gate_nor/gate_nor_2in_1bit/gate_nor_2in.kicad_sch -> ../gate_nor_2in_1bit/gate_nor_2in.kicad_sch
- sheet 2nor6: file ../../modules/gates/gate_nor/gate_nor_2in_1bit/gate_nor_2in.kicad_sch -> ../gate_nor_2in_1bit/gate_nor_2in.kicad_sch
- sheet 2nor7: file ../../modules/gates/gate_nor/gate_nor_2in_1bit/gate_nor_2in.kicad_sch -> ../gate_nor_2in_1bit/gate_nor_2in.kicad_sch
- sheet 2nor8: file ../../modules/gates/gate_nor/gate_nor_2in_1bit/gate_nor_2in.kicad_sch -> ../gate_nor_2in_1bit/gate_nor_2in.kicad_sch
