File: kicad/modules/gates/gate_xor/gate_xor_8bit/gate_xor_8bit.kicad_sch (KiCad schematic)
At the start: 4 parts, among them U701 74HC86, U702 74HC86

Commit message: feat: complete circuit designs for all ALU components
* Designed all gate modules: AND, OR, NOT, NAND, NOR, XOR (1-bit and 8-bit variants)

* Completed multiplexer hierarchy: 2:1, 4:1, and 8:1 8-bit muxes

* Finalized add_sub board schematic and LED panel designs

* Added new board modules: flags, main_control, main_logic

* Updated Logisim top-level ALU circuit

* Note: KiCad directory path errors to be resolved next (iCloud sync issue), then begin PCB routing
Parts:
- renumbered C701 to C2001, C702 to C2002, U701 to U2001, U702 to U2002
Changed lines of the file:
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@@
 		(dnp no)
 		(fields_autoplaced yes)
-		(property "Reference" "U701"
+		(property "Reference" "U2001"
 			(at 194.31 48.2599 0)
 			(effects
@@
 				(path "/3aacef8e-e4d9-474c-bbb9-dab5749c488a/67e1ca7f-32cf-4790-a497-b2e72f19d576/bddc2900-9e93-427b-ba81-f563b34eb8fa"
 					(reference "U101")
+					(unit 5)
+				)
+			)
+			(project ""
+				(path "/9c59990f-2fe5-4da7-bc07-d03b445b1465/6581907b-8185-4495-86c3-6c5c1346d17f"
+					(reference "U2001")
+					(unit 5)
+				)
+				(path "/9c59990f-2fe5-4da7-bc07-d03b445b1465/b047bd69-dc6c-42f6-9708-94c299e28a58"
+					(reference "U701")
 					(unit 5)
 				)
@@
 		(dnp no)
 		(fields_autoplaced yes)
-		(property "Reference" "U702"
+		(property "Reference" "U2002"
 			(at 226.06 48.2599 0)
 			(effects
@@
 				(path "/3aacef8e-e4d9-474c-bbb9-dab5749c488a/67e1ca7f-32cf-4790-a497-b2e72f19d576/bddc2900-9e93-427b-ba81-f563b34eb8fa"
 					(reference "U102")
+					(unit 5)
+				)
+			)
+			(project ""
+				(path "/9c59990f-2fe5-4da7-bc07-d03b445b1465/6581907b-8185-4495-86c3-6c5c1346d17f"
+					(reference "U2002")
+					(unit 5)
+				)
+				(path "/9c59990f-2fe5-4da7-bc07-d03b445b1465/b047bd69-dc6c-42f6-9708-94c299e28a58"
+					(reference "U702")
 					(unit 5)
 				)
@@
 		(dnp no)
 		(fields_autoplaced yes)
-		(property "Reference" "U702"
+		(property "Reference" "U2002"
 			(at 83.5152 127 0)
 			(effects
@@
 				(path "/3aacef8e-e4d9-474c-bbb9-dab5749c488a/67e1ca7f-32cf-4790-a497-b2e72f19d576/bddc2900-9e93-427b-ba81-f563b34eb8fa"
 					(reference "U102")
+					(unit 4)
+				)
+			)
+			(project ""
+				(path "/9c59990f-2fe5-4da7-bc07-d03b445b1465/6581907b-8185-4495-86c3-6c5c1346d17f"
+					(reference "U2002")
+					(unit 4)
+				)
+				(path "/9c59990f-2fe5-4da7-bc07-d03b445b1465/b047bd69-dc6c-42f6-9708-94c299e28a58"
+					(reference "U702")
 					(unit 4)
 				)
@@
 		(dnp no)
 		(fields_autoplaced yes)
-		(property "Reference" "C702"
+		(property "Reference" "C2002"
 			(at 243.84 46.9899 0)
 			(effects
@@
 				(path "/3aacef8e-e4d9-474c-bbb9-dab5749c488a/67e1ca7f-32cf-4790-a497-b2e72f19d576/bddc2900-9e93-427b-ba81-f563b34eb8fa"
 					(reference "C102")
+					(unit 1)
+				)
+			)
+			(project ""
+				(path "/9c59990f-2fe5-4da7-bc07-d03b445b1465/6581907b-8185-4495-86c3-6c5c1346d17f"
+					(reference "C2002")
+					(unit 1)
+				)
+				(path "/9c59990f-2fe5-4da7-bc07-d03b445b1465/b047bd69-dc6c-42f6-9708-94c299e28a58"
+					(reference "C702")
 					(unit 1)
 				)
@@
 		(dnp no)
 		(fields_autoplaced yes)
-		(property "Reference" "U702"
+		(property "Reference" "U2002"
 			(at 83.5152 96.52 0)
 			(effects
@@
 				(path "/3aacef8e-e4d9-474c-bbb9-dab5749c488a/67e1ca7f-32cf-4790-a497-b2e72f19d576/bddc2900-9e93-427b-ba81-f563b34eb8fa"
 					(reference "U102")
+					(unit 2)
+				)
+			)
+			(project ""
+				(path "/9c59990f-2fe5-4da7-bc07-d03b445b1465/6581907b-8185-4495-86c3-6c5c1346d17f"
+					(reference "U2002")
+					(unit 2)
+				)
+				(path "/9c59990f-2fe5-4da7-bc07-d03b445b1465/b047bd69-dc6c-42f6-9708-94c299e28a58"
+					(reference "U702")
 					(unit 2)
 				)
@@
 		(dnp no)
 		(fields_autoplaced yes)
-		(property "Reference" "#PWR0701"
+		(property "Reference" "#PWR02001"
 			(at 187.96 39.37 0)
 			(effects
@@
 				(path "/3aacef8e-e4d9-474c-bbb9-dab5749c488a/67e1ca7f-32cf-4790-a497-b2e72f19d576/bddc2900-9e93-427b-ba81-f563b34eb8fa"
 					(reference "#PWR0102")
+					(unit 1)
+				)
+			)
+			(project ""
+				(path "/9c59990f-2fe5-4da7-bc07-d03b445b1465/6581907b-8185-4495-86c3-6c5c1346d17f"
+					(reference "#PWR02001")
+					(unit 1)
+				)
+				(path "/9c59990f-2fe5-4da7-bc07-d03b445b1465/b047bd69-dc6c-42f6-9708-94c299e28a58"
+					(reference "#PWR0701")
 					(unit 1)
 				)
@@
 		(dnp no)
 		(fields_autoplaced yes)
-		(property "Reference" "#PWR0703"
+		(property "Reference" "#PWR02003"
 			(at 219.71 39.37 0)
 			(effects
@@
 				(path "/3aacef8e-e4d9-474c-bbb9-dab5749c488a/67e1ca7f-32cf-4790-a497-b2e72f19d576/bddc2900-9e93-427b-ba81-f563b34eb8fa"
 					(reference "#PWR0101")
+					(unit 1)
+				)
+			)
+			(project ""
+				(path "/9c59990f-2fe5-4da7-bc07-d03b445b1465/6581907b-8185-4495-86c3-6c5c1346d17f"
+					(reference "#PWR02003")
+					(unit 1)
+				)
+				(path "/9c59990f-2fe5-4da7-bc07-d03b445b1465/b047bd69-dc6c-42f6-9708-94c299e28a58"
+					(reference "#PWR0703")
 					(unit 1)
 				)
@@
 		(dnp no)
 		(fields_autoplaced yes)
-		(property "Reference" "U701"
+		(property "Reference" "U2001"
 			(at 83.5152 35.56 0)
 			(effects
@@
 				(path "/3aacef8e-e4d9-474c-bbb9-dab5749c488a/67e1ca7f-32cf-4790-a497-b2e72f19d576/bddc2900-9e93-427b-ba81-f563b34eb8fa"
 					(reference "U101")
+					(unit 2)
+				)
+			)
+			(project ""
+				(path "/9c59990f-2fe5-4da7-bc07-d03b445b1465/6581907b-8185-4495-86c3-6c5c1346d17f"
+					(reference "U2001")
+					(unit 2)
+				)
+				(path "/9c59990f-2fe5-4da7-bc07-d03b445b1465/b047bd69-dc6c-42f6-9708-94c299e28a58"
+					(reference "U701")
 					(unit 2)
 				)
@@
 		(dnp no)
 		(fields_autoplaced yes)
-		(property "Reference" "U701"
+		(property "Reference" "U2001"
 			(at 83.5152 50.8 0)
 			(effects
@@
 				(path "/3aacef8e-e4d9-474c-bbb9-dab5749c488a/67e1ca7f-32cf-4790-a497-b2e72f19d576/bddc2900-9e93-427b-ba81-f563b34eb8fa"
 					(reference "U101")
+					(unit 3)
+				)
+			)
+			(project ""
+				(path "/9c59990f-2fe5-4da7-bc07-d03b445b1465/6581907b-8185-4495-86c3-6c5c1346d17f"
+					(reference "U2001")
+					(unit 3)
+				)
+				(path "/9c59990f-2fe5-4da7-bc07-d03b445b1465/b047bd69-dc6c-42f6-9708-94c299e28a58"
+					(reference "U701")
 					(unit 3)
 				)
@@
 		(dnp no)
 		(fields_autoplaced yes)
-		(property "Reference" "U701"
+		(property "Reference" "U2001"
 			(at 83.5152 20.32 0)
 			(effects
@@
 				(path "/3aacef8e-e4d9-474c-bbb9-dab5749c488a/67e1ca7f-32cf-4790-a497-b2e72f19d576/bddc2900-9e93-427b-ba81-f563b34eb8fa"
 					(reference "U101")
+					(unit 1)
+				)
+			)
+			(project ""
+				(path "/9c59990f-2fe5-4da7-bc07-d03b445b1465/6581907b-8185-4495-86c3-6c5c1346d17f"
+					(reference "U2001")
+					(unit 1)
+				)
+				(path "/9c59990f-2fe5-4da7-bc07-d03b445b1465/b047bd69-dc6c-42f6-9708-94c299e28a58"
+					(reference "U701")
 					(unit 1)
 				)
@@
 		(dnp no)
 		(fields_autoplaced yes)
-		(property "Reference" "U702"
+		(property "Reference" "U2002"
 			(at 83.5152 81.28 0)
 			(effects
@@
 				(path "/3aacef8e-e4d9-474c-bbb9-dab5749c488a/67e1ca7f-32cf-4790-a497-b2e72f19d576/bddc2900-9e93-427b-ba81-f563b34eb8fa"
 					(reference "U102")
+					(unit 1)
+				)
+			)
+			(project ""
+				(path "/9c59990f-2fe5-4da7-bc07-d03b445b1465/6581907b-8185-4495-86c3-6c5c1346d17f"
+					(reference "U2002")
+					(unit 1)
+				)
+				(path "/9c59990f-2fe5-4da7-bc07-d03b445b1465/b047bd69-dc6c-42f6-9708-94c299e28a58"
+					(reference "U702")
 					(unit 1)
 				)
@@
 		(dnp no)
 		(fields_autoplaced yes)
-		(property "Reference" "U701"
+		(property "Reference" "U2001"
 			(at 83.5152 66.04 0)
 			(effects
@@
 				(path "/3aacef8e-e4d9-474c-bbb9-dab5749c488a/67e1ca7f-32cf-4790-a497-b2e72f19d576/bddc2900-9e93-427b-ba81-f563b34eb8fa"
 					(reference "U101")
+					(unit 4)
+				)
+			)
+			(project ""
+				(path "/9c59990f-2fe5-4da7-bc07-d03b445b1465/6581907b-8185-4495-86c3-6c5c1346d17f"
+					(reference "U2001")
+					(unit 4)
+				)
+				(path "/9c59990f-2fe5-4da7-bc07-d03b445b1465/b047bd69-dc6c-42f6-9708-94c299e28a58"
+					(reference "U701")
 					(unit 4)
 				)
@@
 		(dnp no)
 		(fields_autoplaced yes)
-		(property "Reference" "#PWR0702"
+		(property "Reference" "#PWR02002"
 			(at 187.96 69.85 0)
 			(effects
@@
 				(path "/3aacef8e-e4d9-474c-bbb9-dab5749c488a/67e1ca7f-32cf-4790-a497-b2e72f19d576/bddc2900-9e93-427b-ba81-f563b34eb8fa"
 					(reference "#PWR0103")
+					(unit 1)
+				)
+			)
+			(project ""
+				(path "/9c59990f-2fe5-4da7-bc07-d03b445b1465/6581907b-8185-4495-86c3-6c5c1346d17f"
+					(reference "#PWR02002")
+					(unit 1)
+				)
+				(path "/9c59990f-2fe5-4da7-bc07-d03b445b1465/b047bd69-dc6c-42f6-9708-94c299e28a58"
+					(reference "#PWR0702")
 					(unit 1)
 				)
@@
 		(dnp no)
 		(fields_autoplaced yes)
-		(property "Reference" "U702"
+		(property "Reference" "U2002"
 			(at 83.5152 111.76 0)
 			(effects
@@
 				(path "/3aacef8e-e4d9-474c-bbb9-dab5749c488a/67e1ca7f-32cf-4790-a497-b2e72f19d576/bddc2900-9e93-427b-ba81-f563b34eb8fa"
 					(reference "U102")
+					(unit 3)
+				)
+			)
+			(project ""
+				(path "/9c59990f-2fe5-4da7-bc07-d03b445b1465/6581907b-8185-4495-86c3-6c5c1346d17f"
+					(reference "U2002")
+					(unit 3)
+				)
+				(path "/9c59990f-2fe5-4da7-bc07-d03b445b1465/b047bd69-dc6c-42f6-9708-94c299e28a58"
+					(reference "U702")
 					(unit 3)
 				)
@@
 		(dnp no)
 		(fields_autoplaced yes)
-		(property "Reference" "#PWR0704"
+		(property "Reference" "#PWR02004"
 			(at 219.71 69.85 0)
 			(effects
@@
 				(path "/3aacef8e-e4d9-474c-bbb9-dab5749c488a/67e1ca7f-32cf-4790-a497-b2e72f19d576/bddc2900-9e93-427b-ba81-f563b34eb8fa"
 					(reference "#PWR0104")
+					(unit 1)
+				)
+			)
+			(project ""
+				(path "/9c59990f-2fe5-4da7-bc07-d03b445b1465/6581907b-8185-4495-86c3-6c5c1346d17f"
+					(reference "#PWR02004")
+					(unit 1)
+				)
+				(path "/9c59990f-2fe5-4da7-bc07-d03b445b1465/b047bd69-dc6c-42f6-9708-94c299e28a58"
+					(reference "#PWR0704")
 					(unit 1)
 				)
@@
 		(dnp no)
 		(fields_autoplaced yes)
-		(property "Reference" "C701"
+		(property "Reference" "C2001"
 			(at 175.26 46.9899 0)
 			(effects
@@
 					(unit 1)
 				)
+			)
+			(project ""
+				(path "/9c59990f-2fe5-4da7-bc07-d03b445b1465/6581907b-8185-4495-86c3-6c5c1346d17f"
+					(reference "C2001")
+					(unit 1)
+				)
+				(path "/9c59990f-2fe5-4da7-bc07-d03b445b1465/b047bd69-dc6c-42f6-9708-94c299e28a58"
+					(reference "C701")
+					(unit 1)
+				)

Commit message: Fix KiCad file paths and complete core circuit design
- Fixed file path errors across all KiCad schematics and projects
- Completed core circuit designs:
  * Adder and subtractor modules (adder2, adder8)
  * LED panels (led_panel_1) with display circuits
  * Flag LED circuits for status indicators
  * All dependent logic gate modules (AND, OR, NOT, NAND, NOR, XOR)
  * All multiplexer modules (2:1, 4:1, 8:1, 8-bit)
  * Main control board schematics
  * Flags board schematics
- Updated .gitignore to exclude KiCad backups, cache files, and lock files
- Ready for pin placement and routing of control buses, power rails, and inter-board signals
Parts:
- renumbered C2001 to C701, C2002 to C702, U2001 to U701, U2002 to U702
Changed lines of the file:
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@@
 		(dnp no)
 		(fields_autoplaced yes)
-		(property "Reference" "U2001"
+		(property "Reference" "U701"
 			(at 194.31 48.2599 0)
 			(effects
@@
 		(dnp no)
 		(fields_autoplaced yes)
-		(property "Reference" "U2002"
+		(property "Reference" "U702"
 			(at 226.06 48.2599 0)
 			(effects
@@
 		(dnp no)
 		(fields_autoplaced yes)
-		(property "Reference" "U2002"
+		(property "Reference" "U702"
 			(at 83.5152 127 0)
 			(effects
@@
 		(dnp no)
 		(fields_autoplaced yes)
-		(property "Reference" "C2002"
+		(property "Reference" "C702"
 			(at 243.84 46.9899 0)
 			(effects
@@
 		(dnp no)
 		(fields_autoplaced yes)
-		(property "Reference" "U2002"
+		(property "Reference" "U702"
 			(at 83.5152 96.52 0)
 			(effects
@@
 		(dnp no)
 		(fields_autoplaced yes)
-		(property "Reference" "#PWR02001"
+		(property "Reference" "#PWR0701"
 			(at 187.96 39.37 0)
 			(effects
@@
 		(dnp no)
 		(fields_autoplaced yes)
-		(property "Reference" "#PWR02003"
+		(property "Reference" "#PWR0703"
 			(at 219.71 39.37 0)
 			(effects
@@
 		(dnp no)
 		(fields_autoplaced yes)
-		(property "Reference" "U2001"
+		(property "Reference" "U701"
 			(at 83.5152 35.56 0)
 			(effects
@@
 		(dnp no)
 		(fields_autoplaced yes)
-		(property "Reference" "U2001"
+		(property "Reference" "U701"
 			(at 83.5152 50.8 0)
 			(effects
@@
 		(dnp no)
 		(fields_autoplaced yes)
-		(property "Reference" "U2001"
+		(property "Reference" "U701"
 			(at 83.5152 20.32 0)
 			(effects
@@
 		(dnp no)
 		(fields_autoplaced yes)
-		(property "Reference" "U2002"
+		(property "Reference" "U702"
 			(at 83.5152 81.28 0)
 			(effects
@@
 		(dnp no)
 		(fields_autoplaced yes)
-		(property "Reference" "U2001"
+		(property "Reference" "U701"
 			(at 83.5152 66.04 0)
 			(effects
@@
 		(dnp no)
 		(fields_autoplaced yes)
-		(property "Reference" "#PWR02002"
+		(property "Reference" "#PWR0702"
 			(at 187.96 69.85 0)
 			(effects
@@
 		(dnp no)
 		(fields_autoplaced yes)
-		(property "Reference" "U2002"
+		(property "Reference" "U702"
 			(at 83.5152 111.76 0)
 			(effects
@@
 		(dnp no)
 		(fields_autoplaced yes)
-		(property "Reference" "#PWR02004"
+		(property "Reference" "#PWR0704"
 			(at 219.71 69.85 0)
 			(effects
@@
 		(dnp no)
 		(fields_autoplaced yes)
-		(property "Reference" "C2001"
+		(property "Reference" "C701"
 			(at 175.26 46.9899 0)
 			(effects
