File: kicad/modules/mux/mux_8to1_8bit/mux_8to1_8bit.kicad_sch (KiCad schematic)
At the start: 0 parts

Commit message: feat: complete circuit designs for all ALU components
* Designed all gate modules: AND, OR, NOT, NAND, NOR, XOR (1-bit and 8-bit variants)

* Completed multiplexer hierarchy: 2:1, 4:1, and 8:1 8-bit muxes

* Finalized add_sub board schematic and LED panel designs

* Added new board modules: flags, main_control, main_logic

* Updated Logisim top-level ALU circuit

* Note: KiCad directory path errors to be resolved next (iCloud sync issue), then begin PCB routing
Other:
- sheet 2to1mux: file ../mux_2to1_8bit/mux_2to1_8bit.kicad_sch -> ../../modules/mux/mux_2to1_8bit/mux_2to1_8bit.kicad_sch
- sheet 4to1mux1: file ../mux_4to1_8bit/mux_4to1_8bit.kicad_sch -> ../../modules/mux/mux_4to1_8bit/mux_4to1_8bit.kicad_sch
- sheet 4to1mux2: file ../mux_4to1_8bit/mux_4to1_8bit.kicad_sch -> ../../modules/mux/mux_4to1_8bit/mux_4to1_8bit.kicad_sch
Changed lines of the file:
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@@
 			)
 		)
-		(property "Sheetfile" "../mux_4to1_8bit/mux_4to1_8bit.kicad_sch"
+		(property "Sheetfile" "../../modules/mux/mux_4to1_8bit/mux_4to1_8bit.kicad_sch"
 			(at 52.07 175.8446 0)
 			(effects
@@
 				(path "/c9479498-7c42-47b2-8dd7-3cbf94b88bd8"
 					(page "3")
+				)
+			)
+			(project ""
+				(path "/18b29530-70df-469e-af7f-bd82f36b8ceb"
+					(page "")
+				)
+			)
+			(project "main_logic"
+				(path "/9c59990f-2fe5-4da7-bc07-d03b445b1465/18b29530-70df-469e-af7f-bd82f36b8ceb"
+					(page "19")
 				)
 			)
@@
 			)
 		)
-		(property "Sheetfile" "../mux_2to1_8bit/mux_2to1_8bit.kicad_sch"
+		(property "Sheetfile" "../../modules/mux/mux_2to1_8bit/mux_2to1_8bit.kicad_sch"
 			(at 160.02 125.6796 0)
 			(effects
@@
 				(path "/c9479498-7c42-47b2-8dd7-3cbf94b88bd8"
 					(page "4")
+				)
+			)
+			(project ""
+				(path "/18b29530-70df-469e-af7f-bd82f36b8ceb"
+					(page "")
+				)
+			)
+			(project "main_logic"
+				(path "/9c59990f-2fe5-4da7-bc07-d03b445b1465/18b29530-70df-469e-af7f-bd82f36b8ceb"
+					(page "21")
 				)
 			)
@@
 			)
 		)
-		(property "Sheetfile" "../mux_4to1_8bit/mux_4to1_8bit.kicad_sch"
+		(property "Sheetfile" "../../modules/mux/mux_4to1_8bit/mux_4to1_8bit.kicad_sch"
 			(at 52.07 90.7546 0)
 			(effects
@@
 				)
 			)
+			(project ""
+				(path "/18b29530-70df-469e-af7f-bd82f36b8ceb"
+					(page "")
+				)
+			)
+			(project "main_logic"
+				(path "/9c59990f-2fe5-4da7-bc07-d03b445b1465/18b29530-70df-469e-af7f-bd82f36b8ceb"
+					(page "18")
+				)
+			)
 		)
 	)
-	(sheet_instances
-		(path "/"
-			(page "1")
-		)
-	)
-	(embedded_fonts no)
 )

Commit message: Fix KiCad file paths and complete core circuit design
- Fixed file path errors across all KiCad schematics and projects
- Completed core circuit designs:
  * Adder and subtractor modules (adder2, adder8)
  * LED panels (led_panel_1) with display circuits
  * Flag LED circuits for status indicators
  * All dependent logic gate modules (AND, OR, NOT, NAND, NOR, XOR)
  * All multiplexer modules (2:1, 4:1, 8:1, 8-bit)
  * Main control board schematics
  * Flags board schematics
- Updated .gitignore to exclude KiCad backups, cache files, and lock files
- Ready for pin placement and routing of control buses, power rails, and inter-board signals
Other:
- sheet 2to1mux: file ../../modules/mux/mux_2to1_8bit/mux_2to1_8bit.kicad_sch -> ../mux_2to1_8bit/mux_2to1_8bit.kicad_sch
- sheet 4to1mux1: file ../../modules/mux/mux_4to1_8bit/mux_4to1_8bit.kicad_sch -> ../mux_4to1_8bit/mux_4to1_8bit.kicad_sch
- sheet 4to1mux2: file ../../modules/mux/mux_4to1_8bit/mux_4to1_8bit.kicad_sch -> ../mux_4to1_8bit/mux_4to1_8bit.kicad_sch
Changed lines of the file:
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@@
 			)
 		)
-		(property "Sheetfile" "../../modules/mux/mux_4to1_8bit/mux_4to1_8bit.kicad_sch"
+		(property "Sheetfile" "../mux_4to1_8bit/mux_4to1_8bit.kicad_sch"
 			(at 52.07 175.8446 0)
 			(effects
@@
 			(project ""
 				(path "/18b29530-70df-469e-af7f-bd82f36b8ceb"
-					(page "")
+					(page "#")
 				)
 			)
@@
 			)
 		)
-		(property "Sheetfile" "../../modules/mux/mux_2to1_8bit/mux_2to1_8bit.kicad_sch"
+		(property "Sheetfile" "../mux_2to1_8bit/mux_2to1_8bit.kicad_sch"
 			(at 160.02 125.6796 0)
 			(effects
@@
 			(project ""
 				(path "/18b29530-70df-469e-af7f-bd82f36b8ceb"
-					(page "")
+					(page "#")
 				)
 			)
@@
 			)
 		)
-		(property "Sheetfile" "../../modules/mux/mux_4to1_8bit/mux_4to1_8bit.kicad_sch"
+		(property "Sheetfile" "../mux_4to1_8bit/mux_4to1_8bit.kicad_sch"
 			(at 52.07 90.7546 0)
 			(effects
@@
 			(project ""
 				(path "/18b29530-70df-469e-af7f-bd82f36b8ceb"
-					(page "")
-				)
-			)
+					(page "#")
+				)
+			)
